File: pcb/power_out.kicad_sch (KiCad schematic)
At the start: 5 parts, among them J6 MKDS 3.5mm, Q1 PSMN1R2-30YLC, U1 MCP14A0302

Commit message: work on PCB: line out + power done ; removed amplifier from board
Parts:
- added D3: SS16_R2_00001 1A, 42V, Diode_SMD:D_SMA, symbol Device:D_Schottky
- renumbered Q1 to Q2
Connections:
- net +24V: now also D3.1 (K)
- net at J6.2 (Pin_2), J6.2 (Pin_2), Q2.5 (D): now also D3.2 (A)
Changed lines of the file:
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@@
   (junction (at 134.62 91.44) (diameter 0) (color 0 0 0 0)
   )
+  (junction (at 185.42 87.63) (diameter 0) (color 0 0 0 0)
+  )
   (junction (at 158.75 92.71) (diameter 0) (color 0 0 0 0)
   )
   (junction (at 158.75 90.17) (diameter 0) (color 0 0 0 0)
   )
+  (junction (at 185.42 95.25) (diameter 0) (color 0 0 0 0)
+  )
   (wire (pts (xy 158.75 92.71) (xy 158.75 95.25))
     (stroke (width 0) (type default))
@@
     (stroke (width 0) (type default))
   )
-  (wire (pts (xy 158.75 87.63) (xy 194.31 87.63))
+  (wire (pts (xy 158.75 87.63) (xy 185.42 87.63))
+    (stroke (width 0) (type default))
+  )
+  (wire (pts (xy 185.42 87.63) (xy 194.31 87.63))
     (stroke (width 0) (type default))
   )
@@
     (stroke (width 0) (type default))
   )
-  (wire (pts (xy 158.75 95.25) (xy 194.31 95.25))
+  (wire (pts (xy 158.75 95.25) (xy 185.42 95.25))
     (stroke (width 0) (type default))
   )
@@
   )
   (wire (pts (xy 109.22 95.25) (xy 115.57 95.25))
+    (stroke (width 0) (type default))
+  )
+  (wire (pts (xy 185.42 95.25) (xy 194.31 95.25))
     (stroke (width 0) (type default))
   )
@@
   (symbol (lib_id "power:GND") (at 142.24 91.44 90) (unit 1)
     (in_bom yes) (on_board yes) (dnp no) (fields_autoplaced)
-    (property "Reference" "#PWR022" (at 148.59 91.44 0)
+    (property "Reference" "#PWR026" (at 148.59 91.44 0)
       (effects (font (size 1.27 1.27)) hide)
     )
@@
       (project "wakeuplight"
         (path "/f5441fcc-7db8-443c-8d47-1d2e67dbd624/aec5d3bd-aa51-47d6-960a-d96f772ef2bb"
-          (reference "#PWR022") (unit 1)
-        )
-        (path "/f5441fcc-7db8-443c-8d47-1d2e67dbd624/556be24b-5121-4445-bd87-af03e884b8bf"
-          (reference "#PWR027") (unit 1)
+          (reference "#PWR026") (unit 1)
+        )
+        (path "/f5441fcc-7db8-443c-8d47-1d2e67dbd624/556be24b-5121-4445-bd87-af03e884b8bf"
+          (reference "#PWR031") (unit 1)
         )
       )
@@
   (symbol (lib_id "power:+5V") (at 134.62 87.63 0) (unit 1)
     (in_bom yes) (on_board yes) (dnp no) (fields_autoplaced)
-    (property "Reference" "#PWR020" (at 134.62 91.44 0)
+    (property "Reference" "#PWR024" (at 134.62 91.44 0)
       (effects (font (size 1.27 1.27)) hide)
     )
@@
       (project "wakeuplight"
         (path "/f5441fcc-7db8-443c-8d47-1d2e67dbd624/aec5d3bd-aa51-47d6-960a-d96f772ef2bb"
-          (reference "#PWR020") (unit 1)
-        )
-        (path "/f5441fcc-7db8-443c-8d47-1d2e67dbd624/556be24b-5121-4445-bd87-af03e884b8bf"
+          (reference "#PWR024") (unit 1)
+        )
+        (path "/f5441fcc-7db8-443c-8d47-1d2e67dbd624/556be24b-5121-4445-bd87-af03e884b8bf"
+          (reference "#PWR029") (unit 1)
+        )
+      )
+    )
+  )
+  (symbol (lib_id "power:GND") (at 134.62 104.14 0) (unit 1)
+    (in_bom yes) (on_board yes) (dnp no) (fields_autoplaced)
+    (property "Reference" "#PWR025" (at 134.62 110.49 0)
+      (effects (font (size 1.27 1.27)) hide)
+    )
+    (property "Value" "GND" (at 134.62 108.2731 0)
+      (effects (font (size 1.27 1.27)))
+    )
+    (property "Footprint" "" (at 134.62 104.14 0)
+      (effects (font (size 1.27 1.27)) hide)
+    )
+    (property "Datasheet" "" (at 134.62 104.14 0)
+      (effects (font (size 1.27 1.27)) hide)
+    )
+    (pin "1")
+    (instances
+      (project "wakeuplight"
+        (path "/f5441fcc-7db8-443c-8d47-1d2e67dbd624/aec5d3bd-aa51-47d6-960a-d96f772ef2bb"
           (reference "#PWR025") (unit 1)
         )
-      )
-    )
-  )
-  (symbol (lib_id "power:GND") (at 134.62 104.14 0) (unit 1)
-    (in_bom yes) (on_board yes) (dnp no) (fields_autoplaced)
-    (property "Reference" "#PWR021" (at 134.62 110.49 0)
-      (effects (font (size 1.27 1.27)) hide)
-    )
-    (property "Value" "GND" (at 134.62 108.2731 0)
-      (effects (font (size 1.27 1.27)))
-    )
-    (property "Footprint" "" (at 134.62 104.14 0)
-      (effects (font (size 1.27 1.27)) hide)
-    )
-    (property "Datasheet" "" (at 134.62 104.14 0)
-      (effects (font (size 1.27 1.27)) hide)
-    )
-    (pin "1")
-    (instances
-      (project "wakeuplight"
-        (path "/f5441fcc-7db8-443c-8d47-1d2e67dbd624/aec5d3bd-aa51-47d6-960a-d96f772ef2bb"
-          (reference "#PWR021") (unit 1)
-        )
-        (path "/f5441fcc-7db8-443c-8d47-1d2e67dbd624/556be24b-5121-4445-bd87-af03e884b8bf"
-          (reference "#PWR026") (unit 1)
+        (path "/f5441fcc-7db8-443c-8d47-1d2e67dbd624/556be24b-5121-4445-bd87-af03e884b8bf"
+          (reference "#PWR030") (unit 1)
         )
       )
@@
       (project "wakeuplight"
         (path "/f5441fcc-7db8-443c-8d47-1d2e67dbd624/aec5d3bd-aa51-47d6-960a-d96f772ef2bb"
+          (reference "J7") (unit 1)
+        )
+        (path "/f5441fcc-7db8-443c-8d47-1d2e67dbd624/556be24b-5121-4445-bd87-af03e884b8bf"
           (reference "J9") (unit 1)
         )
-        (path "/f5441fcc-7db8-443c-8d47-1d2e67dbd624/556be24b-5121-4445-bd87-af03e884b8bf"
-          (reference "J10") (unit 1)
-        )
       )
     )
@@
   (symbol (lib_id "power:GND") (at 154.94 104.14 0) (unit 1)
     (in_bom yes) (on_board yes) (dnp no) (fields_autoplaced)
-    (property "Reference" "#PWR024" (at 154.94 110.49 0)
+    (property "Reference" "#PWR028" (at 154.94 110.49 0)
       (effects (font (size 1.27 1.27)) hide)
     )
@@
       (project "wakeuplight"
         (path "/f5441fcc-7db8-443c-8d47-1d2e67dbd624/aec5d3bd-aa51-47d6-960a-d96f772ef2bb"
-          (reference "#PWR024") (unit 1)
-        )
-        (path "/f5441fcc-7db8-443c-8d47-1d2e67dbd624/556be24b-5121-4445-bd87-af03e884b8bf"
-          (reference "#PWR029") (unit 1)
+          (reference "#PWR028") (unit 1)
+        )
+        (path "/f5441fcc-7db8-443c-8d47-1d2e67dbd624/556be24b-5121-4445-bd87-af03e884b8bf"
+          (reference "#PWR033") (unit 1)
         )
       )
@@
   (symbol (lib_id "power:+24V") (at 154.94 88.9 0) (unit 1)
     (in_bom yes) (on_board yes) (dnp no) (fields_autoplaced)
-    (property "Reference" "#PWR023" (at 154.94 92.71 0)
+    (property "Reference" "#PWR027" (at 154.94 92.71 0)
       (effects (font (size 1.27 1.27)) hide)
     )
@@
       (project "wakeuplight"
         (path "/f5441fcc-7db8-443c-8d47-1d2e67dbd624/aec5d3bd-aa51-47d6-960a-d96f772ef2bb"
-          (reference "#PWR023") (unit 1)
-        )
-        (path "/f5441fcc-7db8-443c-8d47-1d2e67dbd624/556be24b-5121-4445-bd87-af03e884b8bf"
-          (reference "#PWR028") (unit 1)
+          (reference "#PWR027") (unit 1)
+        )
+        (path "/f5441fcc-7db8-443c-8d47-1d2e67dbd624/556be24b-5121-4445-bd87-af03e884b8bf"
+          (reference "#PWR032") (unit 1)
+        )
+      )
+    )
+  )
+  (symbol (lib_id "Device:D_Schottky") (at 185.42 91.44 270) (unit 1)
+    (in_bom yes) (on_board yes) (dnp no)
+    (property "Reference" "D3" (at 187.452 89.9104 90)
+      (effects (font (size 1.27 1.27)) (justify left))
+    )
+    (property "Value" "SS16_R2_00001 1A, 42V" (at 180.34 97.79 90)
+      (effects (font (size 1.27 1.27)) (justify left))
+    )
+    (property "Footprint" "Diode_SMD:D_SMA" (at 185.42 91.44 0)
+      (effects (font (size 1.27 1.27)) hide)
+    )
+    (property "Datasheet" "~" (at 185.42 91.44 0)
+      (effects (font (size 1.27 1.27)) hide)
+    )
+    (property "OC_MOUSER" "241-SS16_R2_00001" (at 185.42 91.44 90)
+      (effects (font (size 1.27 1.27)) hide)
+    )
+    (pin "1")
+    (pin "2")
+    (instances
+      (project "wakeuplight"
+        (path "/f5441fcc-7db8-443c-8d47-1d2e67dbd624/aec5d3bd-aa51-47d6-960a-d96f772ef2bb"
+          (reference "D3") (unit 1)
+        )
+        (path "/f5441fcc-7db8-443c-8d47-1d2e67dbd624/556be24b-5121-4445-bd87-af03e884b8bf"
+          (reference "D4") (unit 1)
         )
       )
@@
   (symbol (lib_id "Transistor_FET:PSMN5R2-60YL") (at 152.4 99.06 0) (unit 1)
     (in_bom yes) (on_board yes) (dnp no) (fields_autoplaced)
-    (property "Reference" "Q1" (at 157.607 97.8479 0)
+    (property "Reference" "Q2" (at 157.607 97.8479 0)
       (effects (font (size 1.27 1.27)) (justify left))
     )
@@
       (effects (font (size 1.27 1.27)) hide)
     )
-    (property "Datasheet" "https://assets.nexperia.com/documents/data-sheet/PSMN5R2-60YL.pdf" (at 152.4 99.06 0)
+    (property "Datasheet" "https://assets.nexperia.com/documents/data-sheet/PSMN1R2-30YLC.pdf" (at 152.4 99.06 0)
       (effects (font (size 1.27 1.27)) hide)
     )
@@
       (project "wakeuplight"
         (path "/f5441fcc-7db8-443c-8d47-1d2e67dbd624/aec5d3bd-aa51-47d6-960a-d96f772ef2bb"
-          (reference "Q1") (unit 1)
-        )
-        (path "/f5441fcc-7db8-443c-8d47-1d2e67dbd624/556be24b-5121-4445-bd87-af03e884b8bf"
           (reference "Q2") (unit 1)
+        )
+        (path "/f5441fcc-7db8-443c-8d47-1d2e67dbd624/556be24b-5121-4445-bd87-af03e884b8bf"
+          (reference "Q3") (unit 1)
         )
       )
@@
       (project "wakeuplight"
         (path "/f5441fcc-7db8-443c-8d47-1d2e67dbd624/aec5d3bd-aa51-47d6-960a-d96f772ef2bb"
-          (reference "J5") (unit 1)
-        )
-        (path "/f5441fcc-7db8-443c-8d47-1d2e67dbd624/556be24b-5121-4445-bd87-af03e884b8bf"
           (reference "J6") (unit 1)
         )
-      )
+        (path "/f5441fcc-7db8-443c-8d47-1d2e67dbd624/556be24b-5121-4445-bd87-af03e884b8bf"
+          (reference "J8") (unit 1)
+        )
+      )

Commit message: PCB done
Parts:
- U1: OC_MOUSER (none) -> 579-MCP14A0302T-E/MS
Changed lines of the file:
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@@
+      (effects (font (size 1.27 1.27)) hide)
+    )
+    (property "OC_MOUSER" "579-MCP14A0302T-E/MS" (at 124.46 99.06 0)
       (effects (font (size 1.27 1.27)) hide)
     )
