File: pcb/regulator_5v.kicad_sch (KiCad schematic)
At the start: 11 parts, among them U2 LMR16006YQ

Commit message: work on PCB: line out + power done ; removed amplifier from board
Parts:
- R5: footprint Resistor_SMD:R_0805_2012Metric -> Resistor_SMD:R_0402_1005Metric
Changed lines of the file:
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@@
       (effects (font (size 1.27 1.27)) (justify left))
     )
-    (property "Footprint" "Resistor_SMD:R_0805_2012Metric" (at 175.26 97.79 0)
+    (property "Footprint" "Resistor_SMD:R_0402_1005Metric" (at 175.26 97.79 0)
       (effects (font (size 1.27 1.27)) hide)
     )
@@
       (project "wakeuplight"
         (path "/f5441fcc-7db8-443c-8d47-1d2e67dbd624/5a70dd9e-7f38-4000-902e-423cf3bc2c79"
-          (reference "R4") (unit 1)
+          (reference "R9") (unit 1)
         )
       )
@@
       (project "wakeuplight"
         (path "/f5441fcc-7db8-443c-8d47-1d2e67dbd624/5a70dd9e-7f38-4000-902e-423cf3bc2c79"
-          (reference "#PWR036") (unit 1)
+          (reference "#PWR040") (unit 1)
         )
       )
@@
       (effects (font (size 1.27 1.27)))
     )
-    (property "Footprint" "Resistor_SMD:R_0805_2012Metric" (at 120.65 90.17 0)
+    (property "Footprint" "Resistor_SMD:R_0402_1005Metric" (at 120.65 90.17 0)
       (effects (font (size 1.27 1.27)) hide)
     )
@@
       (project "wakeuplight"
         (path "/f5441fcc-7db8-443c-8d47-1d2e67dbd624/5a70dd9e-7f38-4000-902e-423cf3bc2c79"
-          (reference "R3") (unit 1)
+          (reference "R8") (unit 1)
         )
       )
@@
       (project "wakeuplight"
         (path "/f5441fcc-7db8-443c-8d47-1d2e67dbd624/5a70dd9e-7f38-4000-902e-423cf3bc2c79"
-          (reference "#PWR031") (unit 1)
+          (reference "#PWR035") (unit 1)
         )
       )
@@
       (project "wakeuplight"
         (path "/f5441fcc-7db8-443c-8d47-1d2e67dbd624/5a70dd9e-7f38-4000-902e-423cf3bc2c79"
-          (reference "#PWR032") (unit 1)
+          (reference "#PWR036") (unit 1)
         )
       )
@@
       (project "wakeuplight"
         (path "/f5441fcc-7db8-443c-8d47-1d2e67dbd624/5a70dd9e-7f38-4000-902e-423cf3bc2c79"
-          (reference "#FLG03") (unit 1)
+          (reference "#FLG04") (unit 1)
         )
       )
@@
       (effects (font (size 1.27 1.27)) (justify left))
     )
-    (property "Footprint" "Resistor_SMD:R_0805_2012Metric" (at 175.26 105.41 0)
+    (property "Footprint" "Resistor_SMD:R_0402_1005Metric" (at 175.26 105.41 0)
       (effects (font (size 1.27 1.27)) hide)
     )
@@
       (project "wakeuplight"
         (path "/f5441fcc-7db8-443c-8d47-1d2e67dbd624/5a70dd9e-7f38-4000-902e-423cf3bc2c79"
-          (reference "R5") (unit 1)
+          (reference "R10") (unit 1)
         )
       )
@@
       (project "wakeuplight"
         (path "/f5441fcc-7db8-443c-8d47-1d2e67dbd624/5a70dd9e-7f38-4000-902e-423cf3bc2c79"
-          (reference "#PWR033") (unit 1)
+          (reference "#PWR037") (unit 1)
         )
       )
@@
       (project "wakeuplight"
         (path "/f5441fcc-7db8-443c-8d47-1d2e67dbd624/5a70dd9e-7f38-4000-902e-423cf3bc2c79"
-          (reference "D3") (unit 1)
+          (reference "D5") (unit 1)
         )
       )
@@
       (project "wakeuplight"
         (path "/f5441fcc-7db8-443c-8d47-1d2e67dbd624/5a70dd9e-7f38-4000-902e-423cf3bc2c79"
-          (reference "#PWR030") (unit 1)
+          (reference "#PWR034") (unit 1)
         )
       )
@@
       (project "wakeuplight"
         (path "/f5441fcc-7db8-443c-8d47-1d2e67dbd624/5a70dd9e-7f38-4000-902e-423cf3bc2c79"
-          (reference "#PWR035") (unit 1)
+          (reference "#PWR039") (unit 1)
         )
       )
@@
       (project "wakeuplight"
         (path "/f5441fcc-7db8-443c-8d47-1d2e67dbd624/5a70dd9e-7f38-4000-902e-423cf3bc2c79"
-          (reference "#PWR034") (unit 1)
-        )
-      )
+          (reference "#PWR038") (unit 1)
+        )
+      )

Commit message: PCB done
Parts:
- R8: renamed from R5; value 100k -> 200k
- renumbered C3 to C5, C3 to C6, C5 to C7, C7 to C8, C8 to C9, D7 to D5, R5 to R10, R5 to R9, U2 to U3
Connections:
- net ~{SHDN}: now reaches R8.2, U3.4 (~{SHDN})
